File: Main board/Main board.kicad_pcb (KiCad board)
At the start: 4 copper layers, 51 parts, among them J1 TagConnect_TC2030-NL, J2 Conn_01x20_Pin, J3 Conn_01x20_Pin, J4 MEM2080-00-128-00-A_REVA, SW1 SKRKAEE020, U1 STM32U575VGTx, U2 BMI088, U3 MS5607-02BA03, U4 ADXL375BCCZ-RL7, U5 SN74LVC1G32MDBVREP, X1 1XXD32000MBA

Commit message: Changed to single-board architecture
SPI Layout #1. Shared bus close to USB D+-, might be bad for layout later.
Parts:
- removed JP1: SolderJumper_3_Open, Jumper:SolderJumper-3_P2.0mm_Open_TrianglePad1.0x1.5mm
- added C23: 1uF, PCM_JLCPCB:C_0402, F.Cu at (49.8, 102.1)
- added C24: 10uF, PCM_JLCPCB:C_0402, F.Cu at (50.1, 100.2)
- added C25: 10nF, PCM_JLCPCB:C_0402, F.Cu at (17.2, 99.8)
- added C26: 10uF, PCM_JLCPCB:C_0402, F.Cu at (104.5, 102.4)
- added C27: 10uF, PCM_JLCPCB:C_0603, F.Cu at (189.1, 111.8)
- added C28: 22uF, PCM_JLCPCB:C_0603, F.Cu at (174.2, 112.0)
- added C29: 10nF, PCM_JLCPCB:C_0402, F.Cu at (196.5, 108.5)
- added C30: 100nF, PCM_JLCPCB:C_0402, F.Cu at (210.8, 92.3)
- added C31: 10uF, PCM_JLCPCB:C_0603, F.Cu at (194.3, 120.0)
- added C32: 100nF, PCM_JLCPCB:C_0603, F.Cu at (192.6, 120.0)
- added D1: USBLC6-2SC6, EasyEDA:SOT-23-6_L2.9-W1.6-P0.95-LS2.8-BL, F.Cu at (194.4, 98.3)
- added D2: 3V 500mW, EasyEDA:SOD-123_L2.8-W1.8-LS3.7-RD, F.Cu at (211.3, 89.6)
- added D3: 550mV@3A, EasyEDA:SMA_L4.4-W2.6-LS5.0-RD, F.Cu at (193.3, 114.0)
- added J5: Connector, USB-TYPE-C-16P, PCM_JLCPCB:TYPE-C-SMD_HX-TYPE-C-16PIN, F.Cu at (201.1, 98.3)
- added J6: 436500201, molex1x03:CONN_SD-43650-001_02_MOL, F.Cu at (197.3, 116.1)
- added L1: XFL4020-222MEC_C122469, EasyEDA:IND-SMD_L4.0-W4.0_XAL4030-332MEC, F.Cu at (188.8, 106.2)
- added R17: 4.7kΩ, PCM_JLCPCB:R_0402, F.Cu at (52.7, 100.3)
- added R18: 4.7kΩ, PCM_JLCPCB:R_0402, F.Cu at (52.7, 102.1)
- added R19: 4.7kΩ, PCM_JLCPCB:R_0402, F.Cu at (20.0, 97.9)
- added R20: 4.7kΩ, PCM_JLCPCB:R_0402, F.Cu at (20.0, 99.8)
- added R21: 4.7kΩ, PCM_JLCPCB:R_0402, F.Cu at (20.0, 101.6)
- added R22: 5.1kΩ, PCM_JLCPCB:R_0402, F.Cu at (104.5, 104.2)
- added R23: 5.1kΩ, PCM_JLCPCB:R_0402, F.Cu at (104.5, 106.1)
- added R24: 76.8kΩ, PCM_JLCPCB:R_0603, F.Cu at (196.8, 106.9)
- added R25: 26.1kΩ, PCM_JLCPCB:R_0603, F.Cu at (196.8, 109.8)
- added R26: 10kΩ, PCM_JLCPCB:R_0603, F.Cu at (168.6, 119.8)
- added R27: 47kΩ, PCM_JLCPCB:R_0402, F.Cu at (210.8, 94.1)
- added R28: 27kΩ, PCM_JLCPCB:R_0402, F.Cu at (210.8, 96.0)
- added SW2: SKRKAEE020, EasyEDA:SW-SMD_L3.9-W3.0-P4.45, F.Cu at (48.8, 166.5)
- added U6: MMC5983MA, EasyEDA:LGA-16_L3.0-W3.0-P0.50-BL_SQ, F.Cu at (46.2, 101.2)
- added U7: TMP75AIDR - SOIC, EasyEDA:SOIC-8_L4.9-W3.9-P1.27-LS6.0-BL, F.Cu at (24.9, 101.3)
- added U8: STM32G0B1CBTx, Package_QFP:LQFP-48_7x7mm_P0.5mm, F.Cu at (308.5, -65.2)
- added U9: ICM-45686, EasyEDA:LGA-14_L3.0-W2.5-P0.50-TL, F.Cu at (21.0, 83.5)
- C17, C18, C19, R14: moved to F.Cu
- C22: moved to B.Cu
- R15: value 47kΩ -> 22Ω; moved to F.Cu
- R16: value 47kΩ -> 22Ω
- U2: value BMI088 -> TPS62901RPJR; footprint EasyEDA:LGA-16_L4.5-W3.0-P0.50-BL -> TPSnew:QFN_902RPJR_TEX
- moved J3 350.3 mm to (337.2, -96.0)
- moved J2 304.3 mm to (279.2, -98.8)
- moved C12 168.4 mm to (48.0, 190.2)
- moved C13 168.4 mm to (48.0, 192.1)
- moved C14 168.4 mm to (48.0, 193.9)
- moved R10 159.4 mm to (27.8, 176.0)
- moved R11 159.4 mm to (27.8, 177.9)
- moved R12 159.4 mm to (27.8, 179.7)
- moved R13 159.4 mm to (27.8, 181.6)
- moved C15 157.6 mm to (25.0, 172.3)
- moved FB1 157.1 mm to (47.8, 186.8)
- moved R9 154.8 mm to (26.4, 169.4)
- moved C22 151.7 mm to (166.3, 69.0), turned to 90 degrees
- moved C16 151.2 mm to (165.0, 57.7)
- moved C20 146.4 mm to (161.0, 57.7)
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Connections:
- C1 pad 2: GND -> VBAT-
- C10 pad 2: GND -> VBAT-
- C12 pad 2: GND -> VBAT-
- C13 pad 2: GND -> VBAT-
- C14 pad 2: GND -> VBAT-
- C15 pad 2: GND -> VBAT-
- C16 pad 2: GND -> VBAT-
- C17 pad 2: GND -> VBAT-
- C18 pad 2: GND -> VBAT-
- C19 pad 2: GND -> VBAT-
- C2 pad 2: GND -> VBAT-
- C20 pad 2: GND -> VBAT-
- C21 pad 2: GND -> VBAT-
- C22 pad 2: GND -> VBAT-
- C3 pad 2: GND -> VBAT-
- C4 pad 2: GND -> VBAT-
- C5 pad 2: GND -> VBAT-
- C6 pad 2: GND -> VBAT-
- C7 pad 2: GND -> VBAT-
- C8 pad 2: GND -> VBAT-
- C9 pad 2: GND -> VBAT-
- J1 pad 5: GND -> VBAT-
- J4 pad P6: GND -> VBAT-
- R15 pad 1: BMI_ACCEL_CS -> Net-(U1-PB13)
- R15 pad 2: +3V3 -> SPI2_SCLK
- R16 pad 1: BMI_GYRO_CS -> Net-(U1-PB15)
- R16 pad 2: +3V3 -> SPI2_MOSI
- R7 pad 2: GND -> VBAT-
- R8 pad 2: GND -> VBAT-
- SW1 pad 2: GND -> VBAT-
- U1 pad 10: GND -> VBAT-
- U1 pad 15: unconnected-(U1-PC0-Pad15) -> BAT_LEVEL
- U1 pad 19: GND -> VBAT-
- U1 pad 20: GND -> VBAT-
- U1 pad 23: unconnected-(U1-PA0-Pad23) -> UART4_TX
- U1 pad 24: unconnected-(U1-PA1-Pad24) -> UART4_RX
- U1 pad 26: BMI_ACCEL_INT1 -> ICM_INT1
- U1 pad 27: GND -> VBAT-
- U1 pad 29: BMI_ACCEL_INT2 -> ICM_INT2
- U1 pad 30: BMI_GYRO_CS -> ICM_CS
- U1 pad 31: BMI_GYRO_INT1 -> unconnected-(U1-PA6-Pad31)
- U1 pad 32: BMI_GYRO_INT2 -> unconnected-(U1-PA7-Pad32)
- U1 pad 33: BMI_ACCEL_CS -> unconnected-(U1-PC4-Pad33)
- U1 pad 41: unconnected-(U1-PE10-Pad41) -> ICM_INT_1
- U1 pad 42: unconnected-(U1-PE11-Pad42) -> ICM_INT_2
- U1 pad 43: unconnected-(U1-PE12-Pad43) -> ICM_CS
- U1 pad 49: GND -> VBAT-
- U1 pad 51: ADXL_INT2 -> MS5607_CS
- U1 pad 52: ADXL_INT1 -> Net-(U1-PB13)
- U1 pad 53: ADXL_CS -> SPI2_MISO
- U1 pad 54: unconnected-(U1-PB15-Pad54) -> Net-(U1-PB15)
- U1 pad 57: unconnected-(U1-PD10-Pad57) -> ADXL_INT2
- U1 pad 58: unconnected-(U1-PD11-Pad58) -> ADXL_INT1
- U1 pad 59: unconnected-(U1-PD12-Pad59) -> MMC_SCL
- U1 pad 60: unconnected-(U1-PD13-Pad60) -> MMC_SDA
- U1 pad 61: unconnected-(U1-PD14-Pad61) -> ADXL_CS
- U1 pad 68: unconnected-(U1-PA9-Pad68) -> USART1_TX
- U1 pad 69: unconnected-(U1-PA10-Pad69) -> USART1_RX
- U1 pad 74: GND -> VBAT-
- U1 pad 82: unconnected-(U1-PD1-Pad82) -> COCK
- U1 pad 84: unconnected-(U1-PD3-Pad84) -> MISO
- U1 pad 85: unconnected-(U1-PD4-Pad85) -> MOSI
- U1 pad 86: unconnected-(U1-PD5-Pad86) -> USART2_TX
- U1 pad 87: unconnected-(U1-PD6-Pad87) -> USART2_RX
- U1 pad 92: unconnected-(U1-PB6-Pad92) -> TMP_MAIN_SCL
- U1 pad 93: unconnected-(U1-PB7-Pad93) -> TMP_MAIN_SDA
- U1 pad 94: GND -> VBAT-
- U1 pad 99: GND -> VBAT-
- U2 pad 1: BMI_ACCEL_INT2 -> Net-(U2-PG)
- U2 pad 2: unconnected-(U2-NC-Pad2) -> Net-(U2-SW)
- U2 pad 3: +3V3 -> +5V
- U2 pad 4: GND -> VBAT-
- U2 pad 5: BMI_GYRO_CS -> VBAT+
- U2 pad 6: GND -> VBAT+
- U2 pad 7: GND -> Net-(U2-MODE/S-CONF)
- U2 pad 8: SPI1_SCLK -> Net-(U2-SS/TR)
- U2 pad 9: SPI1_MOSI -> Net-(U2-FB/VSET)
- U3 pad 2: GND -> VBAT-
- U3 pad 3: GND -> VBAT-
- U3 pad 6: SPI1_MISO -> SPI2_MISO
- U3 pad 7: SPI1_MOSI -> SPI2_MOSI
- U3 pad 8: SPI1_SCLK -> SPI2_SCLK
- U4 pad 12: SPI1_MISO -> SPI2_MISO
- U4 pad 14: SPI1_SCLK -> SPI2_SCLK
- U4 pad 2: GND -> VBAT-
- U4 pad 4: GND -> VBAT-
- U4 pad 5: GND -> VBAT-
- U5 pad 1: SPI1_MOSI -> SPI2_MOSI
- U5 pad 3: GND -> VBAT-
- X1 pad 1: GND -> VBAT-
- X1 pad 2: GND -> VBAT-
Routing:
- net SPI1_MISO: track 46.1 -> 0.00 mm, vias 3 -> 0
- net SPI1_SCLK: track 40.1 -> 0.00 mm
- net Net-(J4-SHIELD): track 0.00 -> 39.9 mm
- net SPI2_MISO: track 0.00 -> 35.7 mm, vias 0 -> 2
- net SPI1_MOSI: track 28.6 -> 0.00 mm, vias 3 -> 0
- net SPI2_SCLK: track 0.00 -> 26.9 mm
- net SPI2_MOSI: track 0.00 -> 24.5 mm, vias 0 -> 1
- net MS5607_CS: track 4.03 -> 25.2 mm, vias 1 -> 2
- net ADXL_INT1: track 9.49 -> 18.4 mm
- net ADXL_INT2: track 9.00 -> 17.3 mm
- net ADXL_CS: track 24.2 -> 30.9 mm
- net D-: track 0.00 -> 6.52 mm
- net BMI_ACCEL_CS: track 4.84 -> 0.00 mm, vias 2 -> 0
- net BMI_GYRO_INT2: track 4.30 -> 0.00 mm, vias 1 -> 0
- net Net-(C31-Pad1): track 0.00 -> 4.04 mm
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Other:
- board outline added: 117.4 x 84.8 mm

Commit message: Schematics completed + layout
Parts:
- removed C25: 10nF, PCM_JLCPCB:C_0402
- removed J2, J3: Conn_01x20_Pin, Connector_PinHeader_2.54mm:PinHeader_1x20_P2.54mm_Vertical
- removed R19, R20, R21: 4.7kΩ, PCM_JLCPCB:R_0402
- removed U7: TMP75AIDR - SOIC, EasyEDA:SOIC-8_L4.9-W3.9-P1.27-LS6.0-BL
- removed U8: STM32G0B1CBTx, Package_QFP:LQFP-48_7x7mm_P0.5mm
- added BUZZER1: PS1440P02BT, EasyEDA:BUZ-TH_BD14.0-P5.00-D0.7-FD, F.Cu at (140.3, 114.4)
- added C33: 100nF, PCM_JLCPCB:C_0402, F.Cu at (260.8, 148.0)
- added C34: 4.7uF, PCM_JLCPCB:C_0402, B.Cu at (169.5, 78.8)
- added C35: 10uF, PCM_JLCPCB:C_0402, F.Cu at (179.8, 99.1)
- added C36: 10uF, PCM_JLCPCB:C_0402, F.Cu at (184.3, 95.6)
- added CN1: PA001-4P, EasyEDA:CONN-TH_4P-P5.08_PA001-4P, F.Cu at (198.5, 61.5)
- added CN2: PA001-4P, EasyEDA:CONN-TH_4P-P5.08_PA001-4P, F.Cu at (198.2, 84.0)
- added J7: Conn_01x04_Pin, Connector_PinHeader_2.54mm:PinHeader_1x04_P2.54mm_Vertical, F.Cu at (207.4, 133.2)
- added J8: Conn_01x04_Pin, Connector_PinHeader_2.54mm:PinHeader_1x04_P2.54mm_Vertical, F.Cu at (120.8, 91.6)
- added Q1: SI7232DN-T1-GE3, EasyEDA:POWER-1212-8_L3.3-W3.3-P0.66-LS3.3-BL, F.Cu at (186.5, 73.3)
- added Q2: SI7232DN-T1-GE3, EasyEDA:POWER-1212-8_L3.3-W3.3-P0.66-LS3.3-BL, F.Cu at (186.5, 77.9)
- added Q3: SI7232DN-T1-GE3, EasyEDA:POWER-1212-8_L3.3-W3.3-P0.66-LS3.3-BL, F.Cu at (256.8, 149.3)
- added R29: 47kΩ, PCM_JLCPCB:R_0402, F.Cu at (260.8, 149.8)
- added R30: 1kΩ, PCM_JLCPCB:R_0402, B.Cu at (140.3, 111.8)
- added R31: 10kΩ, PCM_JLCPCB:R_0402, F.Cu at (172.5, 69.2)
- added R32: 3.3kΩ, PCM_JLCPCB:R_0402, F.Cu at (204.2, 27.6)
- added R33: 3.3kΩ, PCM_JLCPCB:R_0402, F.Cu at (204.2, 29.5)
- added R34: 3.3kΩ, PCM_JLCPCB:R_0402, F.Cu at (204.2, 31.4)
- added R35: 1kΩ, PCM_JLCPCB:R_0402, F.Cu at (204.2, 33.2)
- added R36: 1kΩ, PCM_JLCPCB:R_0402, F.Cu at (204.2, 35.0)
- added R37: 1kΩ, PCM_JLCPCB:R_0402, F.Cu at (204.2, 36.9)
- added R38: 1kΩ, PCM_JLCPCB:R_0402, F.Cu at (204.2, 38.8)
- added U10: TLV75733PDBV, Package_TO_SOT_SMD:SOT-23-5, F.Cu at (183.2, 98.8)
- added U11: NRVB120VLSFT1G, EasyEDA:SOD-123_L2.7-W1.6-LS3.7-RD-1, F.Cu at (184.9, 105.0)
- added U12: NRVB120VLSFT1G, EasyEDA:SOD-123_L2.7-W1.6-LS3.7-RD-1, F.Cu at (189.0, 103.5)
- C1, C10, C11, C12, C13, C14, C3, C4, C5, C6, C7, C8, C9, FB1, R1, R17, R18, R4, X1: moved to B.Cu
- L1: value XFL4020-222MEC_C122469 -> CKCS4018-1UH/N; footprint EasyEDA:IND-SMD_L4.0-W4.0_XAL4030-332MEC -> EasyEDA:IND-SMD_L4.0-W4.0
- R16: moved to F.Cu
- R2: value 22Ω -> 3.3kΩ
- moved R2 186.5 mm to (204.2, 25.8)
- moved C14 167.8 mm to (182.2, 93.2), turned to 45 degrees
- moved C13 166.4 mm to (180.0, 90.8), turned to -135 degrees
- moved C12 165.1 mm to (179.0, 89.8), turned to -135 degrees
- moved FB1 163.5 mm to (181.0, 92.0), turned to -135 degrees
- moved X1 155.9 mm to (175.5, 96.5), turned to 90 degrees
- moved U9 155.7 mm to (176.0, 69.2), turned to 180 degrees
- moved C10 155.5 mm to (175.5, 99.0), turned to 180 degrees
- moved C11 154.4 mm to (176.0, 93.2), turned to 90 degrees
- moved C17 151.9 mm to (176.5, 66.0), turned to 90 degrees
- moved C30 149.3 mm to (75.3, 29.7)
- moved D2 149.3 mm to (75.8, 27.0)
- moved R27 149.3 mm to (75.3, 31.6)
- moved R28 149.3 mm to (75.3, 33.4)
- moved C19 147.5 mm to (172.5, 67.8), turned to 180 degrees
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Connections:
- J1 pad 3: Net-(J1-~{RESET}) -> nRST
- R15 pad 1: Net-(U1-PB13) -> SPI2_SCLK
- R15 pad 2: SPI2_SCLK -> Net-(U1-PD1)
- R16 pad 1: Net-(U1-PB15) -> SPI2_MOSI
- R16 pad 2: SPI2_MOSI -> Net-(U1-PD4)
- R2 pad 1: Net-(J1-~{RESET}) -> FIRE_B
- R2 pad 2: nRST -> VBAT-
- U1 pad 26: ICM_INT1 -> unconnected-(U1-PA3-Pad26)
- U1 pad 29: ICM_INT2 -> FIRE_A
- U1 pad 30: ICM_CS -> FIRE_B
- U1 pad 31: unconnected-(U1-PA6-Pad31) -> FIRE_C
- U1 pad 32: unconnected-(U1-PA7-Pad32) -> FIRE_D
- U1 pad 43: ICM_CS -> unconnected-(U1-PE12-Pad43)
- U1 pad 47: unconnected-(U1-PB10-Pad47) -> ICM_CS
- U1 pad 48: unconnected-(U1-VCAP-Pad48) -> Net-(U1-VCAP)
- U1 pad 51: MS5607_CS -> unconnected-(U1-PB12-Pad51)
- U1 pad 52: Net-(U1-PB13) -> unconnected-(U1-PB13-Pad52)
- U1 pad 53: SPI2_MISO -> unconnected-(U1-PB14-Pad53)
- U1 pad 54: Net-(U1-PB15) -> unconnected-(U1-PB15-Pad54)
- U1 pad 55: unconnected-(U1-PD8-Pad55) -> USART3_RX
- U1 pad 56: unconnected-(U1-PD9-Pad56) -> USART3_TX
- U1 pad 57: ADXL_INT2 -> unconnected-(U1-PD10-Pad57)
- U1 pad 58: ADXL_INT1 -> unconnected-(U1-PD11-Pad58)
- U1 pad 61: ADXL_CS -> MMC_INT
- U1 pad 67: unconnected-(U1-PA8-Pad67) -> Beeper
- U1 pad 77: unconnected-(U1-PA15-Pad77) -> ADXL_INT1
- U1 pad 81: unconnected-(U1-PD0-Pad81) -> ADXL_CS
- U1 pad 82: COCK -> Net-(U1-PD1)
- U1 pad 84: MISO -> SPI2_MISO
- U1 pad 85: MOSI -> Net-(U1-PD4)
- U1 pad 86: USART2_TX -> unconnected-(U1-PD5-Pad86)
- U1 pad 87: USART2_RX -> unconnected-(U1-PD6-Pad87)
- U1 pad 91: unconnected-(U1-PB5-Pad91) -> MS5607_CS
- U4 pad 9: ADXL_INT2 -> unconnected-(U4-INT2-Pad9)
- U9 pad 9: ICM_INT_2 -> Net-(U9-INT2/FSYNC/CLKIN)
Routing:
- net nRST: track 0.00 -> 42.1 mm
- net Net-(J1-SWCLK): track 0.00 -> 33.3 mm, vias 0 -> 2
- net Net-(J1-SWDIO): track 0.00 -> 32.9 mm, vias 0 -> 1
- net Net-(J1-SWO): track 0.00 -> 26.9 mm
- net SPI2_MISO: track 35.7 -> 17.5 mm, vias 2 -> 0
- net ADXL_INT2: track 17.3 -> 0.00 mm
- net ICM_INT_1: track 0.00 -> 13.9 mm
- net SPI1_MISO: track 0.00 -> 9.91 mm, vias 0 -> 2
- net MMC_INT: track 0.00 -> 9.79 mm
- net MMC_SCL: track 0.00 -> 9.75 mm
- net SPI1_SCLK: track 0.00 -> 9.48 mm
- net MMC_SDA: track 0.00 -> 9.37 mm
- net SPI1_MOSI: track 0.00 -> 9.13 mm, vias 0 -> 2
- net ICM_CS: track 0.00 -> 8.30 mm
- net SPI2_MOSI: track 24.5 -> 17.7 mm, vias 1 -> 2
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
Commit message: Layout V1
Parts:
- removed C15: 100nF, PCM_JLCPCB:C_0402
- added H1: MountingHole_Pad_MP, MountingHole:MountingHole_3.2mm_M3_DIN965_Pad_TopBottom, F.Cu at (205.5, 49.8)
- added H2: MountingHole_Pad_MP, MountingHole:MountingHole_3.2mm_M3_DIN965_Pad_TopBottom, F.Cu at (132.8, 49.0)
- added H3: MountingHole_Pad_MP, MountingHole:MountingHole_3.2mm_M3_DIN965_Pad_TopBottom, F.Cu at (132.8, 122.2)
- added H4: MountingHole_Pad_MP, MountingHole:MountingHole_3.2mm_M3_DIN965_Pad_TopBottom, F.Cu at (206.0, 122.2)
- C33, J4, R22, R23, R27, R28, R8: moved to B.Cu
- R17, R18: moved to F.Cu
- moved R12 170.8 mm to (152.6, 63.2)
- moved R13 161.0 mm to (146.4, 72.8), turned to 180 degrees
- moved R10 159.5 mm to (150.3, 73.9), turned to -90 degrees
- moved R9 158.3 mm to (149.8, 70.2)
- moved R8 157.5 mm to (143.2, 65.1), turned to -90 degrees
- moved R11 156.1 mm to (150.4, 81.4), turned to -90 degrees
- moved R27 147.7 mm to (201.8, 107.7), turned to 90 degrees
- moved R28 144.5 mm to (199.5, 107.3), turned to 180 degrees
- moved SW2 137.6 mm to (169.6, 100.8), turned to 90 degrees
- moved R7 137.2 mm to (169.6, 105.7), turned to -90 degrees
- moved C33 126.1 mm to (139.9, 112.0), turned to 90 degrees
- moved D2 122.9 mm to (180.3, 91.6), turned to 45 degrees
- moved C30 119.5 mm to (177.8, 91.2), turned to 45 degrees
- moved R29 107.6 mm to (159.1, 114.5)
- moved Q3 106.8 mm to (155.6, 115.5), turned to 180 degrees
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Connections:
- J4 pad P4: Net-(J4-VDD) -> +3V3
- R13 pad 1: eMMC_CMD -> SDMMC_CMD
- U1 pad 29: FIRE_A -> FIRE_D
- U1 pad 30: FIRE_B -> FIRE_C
- U1 pad 31: FIRE_C -> unconnected-(U1-PA6-Pad31)
- U1 pad 32: FIRE_D -> FIRE_B
- U1 pad 33: unconnected-(U1-PC4-Pad33) -> FIRE_A
- U1 pad 42: ICM_INT_2 -> unconnected-(U1-PE11-Pad42)
- U1 pad 92: TMP_MAIN_SCL -> unconnected-(U1-PB6-Pad92)
- U1 pad 93: TMP_MAIN_SDA -> unconnected-(U1-PB7-Pad93)
Routing:
- net SDMMC_CLK: track 0.00 -> 58.4 mm, vias 0 -> 1
- net DAT0: track 0.00 -> 58.1 mm, vias 0 -> 1
- net DAT1: track 0.00 -> 58.1 mm, vias 0 -> 1
- net DAT3: track 0.00 -> 55.3 mm, vias 0 -> 3
- net SDMMC_CMD: track 0.00 -> 55.2 mm, vias 0 -> 3
- net DAT2: track 0.00 -> 52.2 mm, vias 0 -> 5
- net USB_DN: track 0.00 -> 40.1 mm, vias 0 -> 2
- net USB_DP: track 0.00 -> 39.5 mm, vias 0 -> 2
- net BAT_LEVEL: track 0.00 -> 37.9 mm, vias 0 -> 1
- net USART1_TX: track 0.00 -> 29.6 mm, vias 0 -> 3
- net USART1_RX: track 0.00 -> 29.3 mm, vias 0 -> 1
- net USART3_TX: track 0.00 -> 27.1 mm
- net USART3_RX: track 0.00 -> 26.2 mm
- net FIRE_A: track 0.00 -> 23.0 mm
- net FIRE_B: track 0.00 -> 22.2 mm
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- added copper zone on B.Cu, net VBAT-
- added copper zone on F.Cu, net VBAT-
Other:
- board size 117.4 x 84.8 mm -> 119.9 x 87.3 mm
- board text added: "TELEMETRY"
- board text added: "UART"

Commit message: Update
Parts:
- removed BUZZER1: PS1440P02BT, EasyEDA:BUZ-TH_BD14.0-P5.00-D0.7-FD
- removed C16, C22, C33: 100nF, PCM_JLCPCB:C_0402
- removed C23: 1uF, PCM_JLCPCB:C_0402
- removed C24, C26, C35, C36: 10uF, PCM_JLCPCB:C_0402
- removed C31: 10uF, PCM_JLCPCB:C_0603
- removed C32: 100nF, PCM_JLCPCB:C_0603
- removed C34: 4.7uF, PCM_JLCPCB:C_0402
- removed J4: MEM2080-00-128-00-A_REVA, SDholder:CONN_MEM2080-00-128-00-A_GCT
- removed J8: Conn_01x04_Pin, Connector_PinHeader_2.54mm:PinHeader_1x04_P2.54mm_Vertical
- removed Q3: SI7232DN-T1-GE3, EasyEDA:POWER-1212-8_L3.3-W3.3-P0.66-LS3.3-BL
- removed R17, R18: 4.7kΩ, PCM_JLCPCB:R_0402
- removed R22, R23: 5.1kΩ, PCM_JLCPCB:R_0402
- removed R27, R29: 47kΩ, PCM_JLCPCB:R_0402
- removed R28: 27kΩ, PCM_JLCPCB:R_0402
- removed R30: 1kΩ, PCM_JLCPCB:R_0402
- removed R5: 22Ω, PCM_JLCPCB:R_0402
- removed R8: 1MΩ, PCM_JLCPCB:R_0402
- removed U10: TLV75733PDBV, Package_TO_SOT_SMD:SOT-23-5
- removed U11, U12: NRVB120VLSFT1G, EasyEDA:SOD-123_L2.7-W1.6-LS3.7-RD-1
- added Card1: TF-015, EasyEDA:TF-SMD_TF-015, F.Cu at (130.4, 126.8)
- added G***: LOGO, LOGO, F.Cu at (125.2, 67.8)
- added J2: Conn_01x02_Pin, Connector_Molex:Molex_Micro-Fit_3.0_43650-0215_1x02_P3.00mm_Vertical, F.Cu at (173.5, 65.0)
- added J3: Conn_01x02_Pin, Connector_Molex:Molex_Micro-Fit_3.0_43650-0215_1x02_P3.00mm_Vertical, F.Cu at (160.2, 65.0)
- added JP1: Jumper_2_Bridged, Diode_SMD:D_0805_2012Metric, F.Cu at (175.7, 124.8)
- C17, C18, C19, C2, C20, C21, C30, R10, R11, R12, R13, R14, R15, R16, R2, R3, R31, R32, R33, R34, R35, R36, R37, R38, R6, R7, R9: moved to B.Cu
- J7: footprint Connector_PinHeader_2.54mm:PinHeader_1x04_P2.54mm_Vertical -> 1x04Molex:CONN_SD-43045-010_04_MOL
- U5: moved to F.Cu
- moved H1 90.6 mm to (116.5, 66.5)
- moved H4 90.2 mm to (116.5, 133.5)
- moved R12 64.4 mm to (138.5, 126.0), turned to -90 degrees
- moved H2 53.7 mm to (183.5, 66.5)
- moved H3 52.0 mm to (183.5, 133.5)
- moved R13 51.6 mm to (134.5, 122.9), turned to 90 degrees
- moved R9 49.4 mm to (126.7, 114.0)
- moved R10 45.4 mm to (124.3, 111.0), turned to 180 degrees
- moved R11 43.9 mm to (142.2, 124.5), turned to 0 degrees
- moved R2 42.9 mm to (168.8, 104.2)
- moved R36 42.9 mm to (168.8, 102.8), turned to 0 degrees
- moved J1 42.3 mm to (148.8, 82.8)
- moved C28 38.4 mm to (173.9, 135.2)
- moved R25 38.2 mm to (177.7, 129.8), turned to 0 degrees
- moved R35 38.2 mm to (168.8, 96.2)
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Connections:
- CN1 pad 2: VBAT+ -> PYRO+
- CN1 pad 4: VBAT+ -> PYRO+
- CN2 pad 1: VBAT+ -> PYRO+
- CN2 pad 3: VBAT+ -> PYRO+
- D3 pad 2: Net-(C31-Pad1) -> PYRO+
- J1 pad 6: Net-(J1-SWO) -> unconnected-(J1-SWO-Pad6)
- J6 pad 1: Net-(C31-Pad1) -> PYRO+
- J7 pad 2: USART1_RX -> VBAT-
- J7 pad 4: VBAT- -> USART1_RX
- Q1 pad 1: VBAT- -> PYRO_GND
- Q1 pad 3: VBAT- -> PYRO_GND
- Q2 pad 1: VBAT- -> PYRO_GND
- Q2 pad 3: VBAT- -> PYRO_GND
- U1 pad 23: UART4_TX -> unconnected-(U1-PA0-Pad23)
- U1 pad 24: UART4_RX -> unconnected-(U1-PA1-Pad24)
- U1 pad 25: unconnected-(U1-PA2-Pad25) -> FIRE_B
- U1 pad 26: unconnected-(U1-PA3-Pad26) -> FIRE_A
- U1 pad 29: FIRE_D -> unconnected-(U1-PA4-Pad29)
- U1 pad 30: FIRE_C -> SPI1_SCLK
- U1 pad 31: unconnected-(U1-PA6-Pad31) -> SPI1_MISO
- U1 pad 32: FIRE_B -> SPI1_MOSI
- U1 pad 33: FIRE_A -> unconnected-(U1-PC4-Pad33)
- U1 pad 40: unconnected-(U1-PE9-Pad40) -> PWM1
- U1 pad 41: ICM_INT_1 -> unconnected-(U1-PE10-Pad41)
- U1 pad 42: unconnected-(U1-PE11-Pad42) -> PWM2
- U1 pad 44: SPI1_SCLK -> unconnected-(U1-PE13-Pad44)
- U1 pad 45: SPI1_MISO -> unconnected-(U1-PE14-Pad45)
- U1 pad 46: SPI1_MOSI -> unconnected-(U1-PE15-Pad46)
- U1 pad 47: ICM_CS -> unconnected-(U1-PB10-Pad47)
- U1 pad 53: unconnected-(U1-PB14-Pad53) -> DAT0
- U1 pad 54: unconnected-(U1-PB15-Pad54) -> DAT1
- U1 pad 55: USART3_RX -> unconnected-(U1-PD8-Pad55)
- U1 pad 56: USART3_TX -> unconnected-(U1-PD9-Pad56)
- U1 pad 61: MMC_INT -> unconnected-(U1-PD14-Pad61)
- U1 pad 65: DAT0 -> unconnected-(U1-PC8-Pad65)
- U1 pad 66: DAT1 -> unconnected-(U1-PC9-Pad66)
- U1 pad 67: Beeper -> MS5607_CS
- U1 pad 68: USART1_TX -> USART1_RX
- U1 pad 69: USART1_RX -> USART1_TX
- U1 pad 77: ADXL_INT1 -> unconnected-(U1-PA15-Pad77)
- U1 pad 78: DAT2 -> unconnected-(U1-PC10-Pad78)
- U1 pad 79: DAT3 -> unconnected-(U1-PC11-Pad79)
- U1 pad 8: unconnected-(U1-PC14-Pad8) -> FIRE_D
- U1 pad 80: SDMMC_CLK -> unconnected-(U1-PC12-Pad80)
- U1 pad 83: SDMMC_CMD -> unconnected-(U1-PD2-Pad83)
- U1 pad 87: unconnected-(U1-PD6-Pad87) -> SDMMC_CLK
- U1 pad 88: unconnected-(U1-PD7-Pad88) -> SDMMC_CMD
- U1 pad 89: SWO -> DAT2
- U1 pad 9: unconnected-(U1-PC15-Pad9) -> FIRE_C
- U1 pad 90: unconnected-(U1-PB4-Pad90) -> DAT3
- U1 pad 91: MS5607_CS -> unconnected-(U1-PB5-Pad91)
Routing:
- net USB_DN: track 40.1 -> 0.00 mm, vias 2 -> 0
- net Net-(J4-SHIELD): track 39.9 -> 0.00 mm
- net USB_DP: track 39.5 -> 0.00 mm, vias 2 -> 0
- net BAT_LEVEL: track 37.9 -> 0.00 mm, vias 1 -> 0
- net PWM1: track 0.00 -> 35.5 mm, vias 0 -> 2
- net Net-(J1-SWO): track 29.9 -> 0.00 mm
- net SPI2_MISO: track 17.5 -> 47.3 mm, vias 0 -> 2
- net PWM2: track 0.00 -> 29.5 mm
- net USART3_TX: track 27.1 -> 0.00 mm
- net USART3_RX: track 26.2 -> 0.00 mm
- net PYRO+: track 0.00 -> 24.4 mm
- net SPI2_SCLK: track 22.6 -> 45.6 mm, vias 0 -> 3
- net MMC_SDA: track 14.6 -> 37.1 mm
- net ADXL_INT1: track 21.6 -> 0.00 mm, vias 2 -> 0
- net MMC_SCL: track 13.5 -> 34.8 mm
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- added copper zone on F.Cu, net Net-(U2-SW)
- added copper zone on F.Cu, net PYRO+
- added copper zone on F.Cu, net PYRO_GND
- added copper zone on In2.Cu, net PYRO_GND
- added copper zone on F.Cu, net VBAT+
- added copper zone on In2.Cu, net VBAT+
- added copper zone on In1.Cu, net VBAT-
Other:
- board size 119.9 x 87.3 mm -> 230.2 x 100.5 mm
- board text added: "By Thanapat Suwanrat"
- board text added: "CURSR-V Flight Computer"
- board text added: "D1+"
- board text added: "D1-"
- board text added: "D2+"
- board text added: "D2-"
- board text added: "GND"
- board text added: "M1+"
- board text added: "M1-"
- board text added: "M2+"
- board text added: "M2-"
- board text added: "PE11"
- board text added: "PE9"
- board text removed: "TELEMETRY"
- board text removed: "UART"
