File: Main board/Main board.kicad_sch (KiCad schematic)
At the start: 0 parts

Commit message: Initial Update
Mainboard schematic update - Added MCU, decoupling, Manual reset, 32MHz TCXO, SD card holder, SWD Tag-connect header, SPI sensors
Mainboard layout update - Initial SPI routings
.ioc update - Initial peripheral setups
Parts:
- added C1: 10uF, PCM_JLCPCB:C_0402, symbol PCM_JLCPCB-Capacitors:0402,10uF
- added C10, C13, C14: 1uF, PCM_JLCPCB:C_0402, symbol PCM_JLCPCB-Capacitors:0402,1uF
- added C11: 100pF, PCM_JLCPCB:C_0402, symbol PCM_JLCPCB-Capacitors:0402,100pF
- added C12, C15, C2, C3, C4, C5, C6, C7, C8, C9: 100nF, PCM_JLCPCB:C_0402, symbol PCM_JLCPCB-Capacitors:0402,100nF
- added FB1: 100R, Capacitor_SMD:C_0402_1005Metric_Pad0.74x0.62mm_HandSolder, symbol Device:FerriteBead
- added J1: TagConnect_TC2030-NL, Connector:Tag-Connect_TC2030-IDC-NL_2x03_P1.27mm_Vertical, symbol Connector:Conn_ARM_SWD_TagConnect_TC2030-NL
- added J2, J3: Conn_01x20_Pin, Connector_PinHeader_2.54mm:PinHeader_1x20_P2.54mm_Vertical, symbol Connector:Conn_01x20_Pin
- added J4: MEM2080-00-128-00-A_REVA, SDholder:CONN_MEM2080-00-128-00-A_GCT, symbol MEM2080-00-128-00-A_REVA:MEM2080-00-128-00-A_REVA
- added JP1: SolderJumper_3_Open, Jumper:SolderJumper-3_P2.0mm_Open_TrianglePad1.0x1.5mm, symbol Jumper:SolderJumper_3_Open
- added R1, R10, R11, R12, R13, R9: 10kΩ, PCM_JLCPCB:R_0402, symbol PCM_JLCPCB-Resistors:0402,10kΩ
- added R2, R3, R4, R5: 22Ω, PCM_JLCPCB:R_0402, symbol PCM_JLCPCB-Resistors:0402,22Ω
- added R7: 100kΩ, PCM_JLCPCB:R_0402, symbol PCM_JLCPCB-Resistors:0402,100kΩ
- added R8: 1MΩ, PCM_JLCPCB:R_0402, symbol PCM_JLCPCB-Resistors:0402,1MΩ
- added SW1: SKRKAEE020, EasyEDA:SW-SMD_L3.9-W3.0-P4.45, symbol EasyEDA:SKRKAEE020
- added U1: STM32U575VGTx, Package_QFP:LQFP-100_14x14mm_P0.5mm, symbol MCU_ST_STM32U5:STM32U575VGTx
- added X1: 1XXD32000MBA, EasyEDA:OSC-SMD_4P-L2.0-W1.6-BL_1XXD, symbol EasyEDA:1XXD32000MBA
Connections:
- new net: C11.1, X1.3 (Output)
- new net: J1.6 (SWO), R5.1
- new net: C15.1, J4.P4 (VDD)
- new net: J1.2 (SWDIO), R4.1
- new net: J4.MNT1 (SHIELD), J4.MNT2 (SHIELD__1), J4.MNT3 (SHIELD__2), J4.MNT4 (SHIELD__3), R8.1
- new net: J1.4 (SWCLK), R3.1
- new net: J1.3 (~{RESET}), R2.1
- new net +3.3VA: C12.1, C13.1, FB1.1, U1.21 (VREF+), U1.22 (VDDA)
- new net +3V3: C1.1, C10.1, C14.1, C3.1, C4.1, C5.1, C6.1, C7.1, C8.1, C9.1, FB1.2, J1.1 (VCC), JP1.3 (B), R1.1, R10.2, R11.2, R12.2, R13.2, R7.1, R9.2, U1.100 (VDD), U1.11 (VDD), U1.28 (VDD), U1.50 (VDD), U1.6 (VBAT), U1.73 (VDDUSB), U1.75 (VDD), X1.4 (VCC)
- new net ADXL_CS: U1.53 (PB14)
- new net ADXL_INT1: U1.52 (PB13)
- new net ADXL_INT2: U1.51 (PB12)
- new net BMI_ACCEL_CS: U1.33 (PC4)
- new net BMI_ACCEL_INT1: U1.26 (PA3)
- new net BMI_ACCEL_INT2: U1.29 (PA4)
- new net BMI_GYRO_CS: U1.30 (PA5)
- new net BMI_GYRO_INT1: U1.31 (PA6)
- new net BMI_GYRO_INT2: U1.32 (PA7)
- new net DAT0: J4.P7 (DAT0), R9.1, U1.65 (PC8)
- new net DAT1: J4.P8 (DAT1), R10.1, U1.66 (PC9)
- new net DAT2: J4.P1 (DAT2), R11.1, U1.78 (PC10)
- new net DAT3: J4.P2 (CD/DAT3), R12.1, U1.79 (PC11)
- new net GND: C1.2, C10.2, C12.2, C13.2, C14.2, C15.2, C2.2, C3.2, C4.2, C5.2, C6.2, C7.2, C8.2, C9.2, J1.5 (GND), J4.P6 (VSS), JP1.1 (A), R7.2, R8.2, SW1.2, U1.10 (VSS), U1.19 (VSSA), U1.20 (VREF-), U1.27 (VSS), U1.49 (VSS), U1.74 (VSS), U1.94 (PH3), U1.99 (VSS), X1.1 (GND), X1.2 (GND)
- new net HSE_IN: C11.2, U1.12 (PH0)
- new net SDMMC_CLK: J4.P5 (CLK), U1.80 (PC12)
- new net SDMMC_CMD: J4.P3 (CMD), U1.83 (PD2)
- new net SPI1_MISO: U1.45 (PE14)
- new net SPI1_MOSI: U1.46 (PE15)
- new net SPI1_SCLK: U1.44 (PE13)
- new net SWCLK: R3.2, U1.76 (PA14)
- new net SWDIO: R4.2, U1.72 (PA13)
- new net SWO: R5.2, U1.89 (PB3)
- new net USB_DN: U1.70 (PA11)
- new net USB_DP: U1.71 (PA12)
- new net eMMC_CMD: R13.1
- new net nRST: C2.1, R1.2, R2.2, SW1.1, U1.14 (NRST)
- no-connect marks 0 -> 4
Other:
- added sheet Sensors (untitled.kicad_sch)
- note added: "BOOT0 switch"
- note added: "Debugging"
- note added: "MCU Power and Decoupling"
- note added: "Manual reset"
- note added: "SD Card slot"
- note added: "STM32U5"
- note added: "TCXO"

Commit message: Changed to single-board architecture
SPI Layout #1. Shared bus close to USB D+-, might be bad for layout later.
Parts:
- removed JP1: SolderJumper_3_Open, Jumper:SolderJumper-3_P2.0mm_Open_TrianglePad1.0x1.5mm, symbol Jumper:SolderJumper_3_Open
- added C26: 10uF, PCM_JLCPCB:C_0402, symbol PCM_JLCPCB-Capacitors:0402,10uF
- added C27: 10uF, PCM_JLCPCB:C_0603, symbol PCM_JLCPCB-Capacitors:0603,10uF,(2)
- added C28: 22uF, PCM_JLCPCB:C_0603, symbol PCM_JLCPCB-Capacitors:0603,22uF
- added C29: 10nF, PCM_JLCPCB:C_0402, symbol PCM_JLCPCB-Capacitors:0402,10nF
- added C30: 100nF, PCM_JLCPCB:C_0402, symbol PCM_JLCPCB-Capacitors:0402,100nF
- added C31: 10uF, PCM_JLCPCB:C_0603, symbol PCM_JLCPCB-Capacitors:0603,10uF
- added C32: 100nF, PCM_JLCPCB:C_0603, symbol PCM_JLCPCB-Capacitors:0603,100nF
- added D1: USBLC6-2SC6, EasyEDA:SOT-23-6_L2.9-W1.6-P0.95-LS2.8-BL, symbol EasyEDA:USBLC6-2SC6
- added D2: 3V 500mW, EasyEDA:SOD-123_L2.8-W1.8-LS3.7-RD, symbol EasyEDA:MMSZ4683T1G
- added D3: 550mV@3A, EasyEDA:SMA_L4.4-W2.6-LS5.0-RD, symbol EasyEDA:SS34_C466502
- added J5: Connector, USB-TYPE-C-16P, PCM_JLCPCB:TYPE-C-SMD_HX-TYPE-C-16PIN, symbol PCM_JLCPCB-Extended:Connector, USB-TYPE-C-16P
- added J6: 436500201, molex1x03:CONN_SD-43650-001_02_MOL, symbol molex1x03:436500201
- added L1: XFL4020-222MEC_C122469, EasyEDA:IND-SMD_L4.0-W4.0_XAL4030-332MEC, symbol EasyEDA:XFL4020-222MEC_C122469
- added R15, R16: 22Ω, PCM_JLCPCB:R_0402, symbol PCM_JLCPCB-Resistors:0402,22Ω
- added R22, R23: 5.1kΩ, PCM_JLCPCB:R_0402, symbol PCM_JLCPCB-Resistors:0402,5.1kΩ
- added R24: 76.8kΩ, PCM_JLCPCB:R_0603, symbol PCM_JLCPCB-Resistors:0603,1.1kΩ
- added R25: 26.1kΩ, PCM_JLCPCB:R_0603, symbol PCM_JLCPCB-Resistors:0603,1.1kΩ
- added R26: 10kΩ, PCM_JLCPCB:R_0603, symbol PCM_JLCPCB-Resistors:0603,10kΩ
- added R27: 47kΩ, PCM_JLCPCB:R_0402, symbol PCM_JLCPCB-Resistors:0402,47kΩ
- added R28: 27kΩ, PCM_JLCPCB:R_0402, symbol PCM_JLCPCB-Resistors:0402,27kΩ
- added SW2: SKRKAEE020, EasyEDA:SW-SMD_L3.9-W3.0-P4.45, symbol EasyEDA:SKRKAEE020
- added U2: TPS62901RPJR, QFN_902RPJR_TEX, symbol TPS62901RPJR:TPS62901RPJR
- added U8: STM32G0B1CBTx, Package_QFP:LQFP-48_7x7mm_P0.5mm, symbol MCU_ST_STM32G0:STM32G0B1CBTx
Connections:
- net BMI_GYRO_CS is gone; now on net ICM_CS: U1.30 (PA5)
- net +3V3: now also SW2.1
- net ADXL_CS: now also U1.61 (PD14); no longer U1.53 (PB14)
- net ADXL_INT1: now also U1.58 (PD11); no longer U1.52 (PB13)
- net ADXL_INT2: now also U1.57 (PD10); no longer U1.51 (PB12)
- net GND: now also C26.2, C27.2, C28.2, C29.2, C30.2, C31.2, C32.2, D1.2, D2.2 (A), J6.2, R22.2, R23.2, R24.1, R25.2, R28.2, SW2.2, U2.4 (GND)
- net USB_DN: now also D1.4
- net USB_DP: now also D1.6
- net BAT_LEVEL: now reaches U1.15 (PC0)
- net BAT_LEVEL: now also C30.1, D2.1 (C), R27.2, R28.1
- net UART4_TX: now reaches U1.23 (PA0)
- net UART4_RX: now reaches U1.24 (PA1)
- net ICM_INT_1: now reaches U1.41 (PE10)
- net ICM_INT_2: now reaches U1.42 (PE11)
- net ICM_CS: now reaches U1.43 (PE12)
- net at U1.54 (PB15): now also R16.1
- net MMC_SCL: now reaches U1.59 (PD12)
- net MMC_SDA: now reaches U1.60 (PD13)
- net USART1_TX: now reaches U1.68 (PA9)
- net USART1_RX: now reaches U1.69 (PA10)
- net COCK: now reaches U1.82 (PD1)
- net MISO: now reaches U1.84 (PD3)
- net MOSI: now reaches U1.85 (PD4)
- net USART2_TX: now reaches U1.86 (PD5)
- net USART2_RX: now reaches U1.87 (PD6)
- net TMP_MAIN_SCL: now reaches U1.92 (PB6)
- net TMP_MAIN_SDA: now reaches U1.93 (PB7)
- net BMI_ACCEL_CS: no longer names the net of U1.33 (PC4)
- net BMI_ACCEL_INT1 renamed ICM_INT1
- net BMI_ACCEL_INT2 renamed ICM_INT2
- net BMI_GYRO_INT1: no longer names the net of U1.31 (PA6)
- net BMI_GYRO_INT2: no longer names the net of U1.32 (PA7)
- new net: C31.1, C32.1, D3.2, J6.1
- new net: C29.1, U2.8 (SS/TR)
- new net: J5.A12B1 (GND), J5.B12A1 (GND)
- new net: J5.A5 (CC1), R22.1
- new net: J5.B5 (CC2), R23.1
- new net: R26.2, U2.1 (PG)
- new net: L1.2, U2.2 (SW)
- new net: R25.1, U2.7 (MODE/S-CONF)
- new net: R24.2, U2.9 (FB/VSET)
- new net: R15.1, U1.52 (PB13)
- new net +5V: C28.1, L1.1, R26.1, U2.3 (VOS)
- new net D+: D1.1, J5.A6 (D+), J5.B6 (D+)
- new net D-: D1.3, J5.A7 (D-), J5.B7 (D-)
- new net MS5607_CS: U1.51 (PB12)
- new net SPI2_MISO: U1.53 (PB14)
- new net SPI2_MOSI: R16.2
- new net SPI2_SCLK: R15.2
- new net VBAT+: C27.1, D3.1, R27.1, U2.5 (EN), U2.6 (VIN)
- new net VBUS: C26.1, D1.5, J5.A9B4 (VBUS), J5.B9A4 (VBUS)
- no-connect marks 4 -> 6
Other:
- note added: "5V Buck"
- note added: "8.4V Max"
- note added: "Battery Connector"
- note added: "Divider circuit for ADC"
- note added: "Drops to 3.065V at Vin = 8.4V"
- note added: "For 5V output (From datasheet table)"
- note added: "TO ADC"
- note added: "USB + ESD diodes"
- moved on the sheet: J2, J3, R7

Commit message: Schematics completed + layout
Parts:
- removed J2, J3: Conn_01x20_Pin, Connector_PinHeader_2.54mm:PinHeader_1x20_P2.54mm_Vertical, symbol Connector:Conn_01x20_Pin
- removed L1: XFL4020-222MEC_C122469, EasyEDA:IND-SMD_L4.0-W4.0_XAL4030-332MEC, symbol EasyEDA:XFL4020-222MEC_C122469
- removed R2: 22Ω, PCM_JLCPCB:R_0402, symbol PCM_JLCPCB-Resistors:0402,22Ω
- removed U8: STM32G0B1CBTx, Package_QFP:LQFP-48_7x7mm_P0.5mm, symbol MCU_ST_STM32G0:STM32G0B1CBTx
- added BUZZER1: PS1440P02BT, EasyEDA:BUZ-TH_BD14.0-P5.00-D0.7-FD, symbol EasyEDA:PS1440P02BT
- added C33: 100nF, PCM_JLCPCB:C_0402, symbol PCM_JLCPCB-Capacitors:0402,100nF
- added C34: 4.7uF, PCM_JLCPCB:C_0402, symbol PCM_JLCPCB-Capacitors:0402,4.7uF
- added C35, C36: 10uF, PCM_JLCPCB:C_0402, symbol PCM_JLCPCB-Capacitors:0402,10uF
- added CN1, CN2: PA001-4P, EasyEDA:CONN-TH_4P-P5.08_PA001-4P, symbol EasyEDA:PA001-4P
- added J7, J8: Conn_01x04_Pin, Connector_PinHeader_2.54mm:PinHeader_1x04_P2.54mm_Vertical, symbol Connector:Conn_01x04_Pin
- added L1: CKCS4018-1UH/N, EasyEDA:IND-SMD_L4.0-W4.0, symbol EasyEDA:CKCS4018-1UH_N
- added Q1, Q2, Q3: SI7232DN-T1-GE3, EasyEDA:POWER-1212-8_L3.3-W3.3-P0.66-LS3.3-BL, symbol EasyEDA:SI7232DN-T1-GE3
- added R2, R32, R33, R34: 3.3kΩ, PCM_JLCPCB:R_0402, symbol PCM_JLCPCB-Resistors:0402,3.3kΩ
- added R29: 47kΩ, PCM_JLCPCB:R_0402, symbol PCM_JLCPCB-Resistors:0402,47kΩ
- added R30, R35, R36, R37, R38: 1kΩ, PCM_JLCPCB:R_0402, symbol PCM_JLCPCB-Resistors:0402,1kΩ
- added U10: TLV75733PDBV, Package_TO_SOT_SMD:SOT-23-5, symbol Regulator_Linear:TLV75733PDBV
- added U11, U12: NRVB120VLSFT1G, EasyEDA:SOD-123_L2.7-W1.6-LS3.7-RD-1, symbol EasyEDA:NRVB120VLSFT1G
Connections:
- net MISO is gone; now on net SPI2_MISO: U1.84 (PD3)
- net +3V3: now also C35.1, J7.1 (Pin_1), J8.1 (Pin_1), U10.5 (OUT)
- net +5V: now also L1.1, U12.2 (A)
- net ADXL_CS: now also U1.81 (PD0); no longer U1.61 (PD14)
- net ADXL_INT1: now also U1.77 (PA15); no longer U1.58 (PD11)
- net GND: now also C33.2, C34.2, C35.2, C36.2, J7.4 (Pin_4), J8.4 (Pin_4), Q1.1 (S1), Q1.3 (S2), Q2.1 (S1), Q2.3 (S2), Q3.3 (S2), R2.2, R29.2, R32.2, R33.2, R34.2, U10.2 (GND)
- net ICM_CS: now also U1.47 (PB10); no longer U1.30 (PA5), U1.43 (PE12)
- net MS5607_CS: now also U1.91 (PB5); no longer U1.51 (PB12)
- net SPI2_MISO: no longer U1.53 (PB14)
- net SPI2_MOSI: now also R16.1; no longer R16.2
- net SPI2_SCLK: now also R15.1; no longer R15.2
- net USART1_RX: now also J7.2 (Pin_2)
- net USART1_TX: now also J7.3 (Pin_3)
- net VBAT+: now also CN1.2, CN1.4, CN2.1, CN2.3
- net VBUS: now also U11.2 (A)
- net nRST: now also J1.3 (~{RESET})
- net at U2.2 (SW): now also L1.2
- net at U1.54 (PB15): no longer R16.1
- net FIRE_C: now reaches U1.31 (PA6)
- net FIRE_C: now also R34.1, R37.1
- net FIRE_D: now reaches U1.32 (PA7)
- net FIRE_D: now also R33.1, R38.1
- net at U1.48 (VCAP): now also C34.1
- net at U1.52 (PB13): no longer R15.1
- net USART3_RX: now reaches U1.55 (PD8)
- net USART3_RX: now also J8.2 (Pin_2)
- net USART3_TX: now reaches U1.56 (PD9)
- net USART3_TX: now also J8.3 (Pin_3)
- net Beeper: now reaches U1.67 (PA8)
- net Beeper: now also Q3.4 (G2), R29.1
- net ADXL_INT2: no longer names the net of U1.57 (PD10)
- net COCK: no longer names the net of U1.82 (PD1)
- net COCK: now also R15.2
- net ICM_INT1: no longer names the net of U1.26 (PA3)
- net ICM_INT2 renamed FIRE_A
- net FIRE_A: now also R32.1, R35.1
- net MOSI: no longer names the net of U1.85 (PD4)
- net MOSI: now also R16.2
- net TMP_MAIN_SCL: no longer names the net of U1.92 (PB6)
- net TMP_MAIN_SDA: no longer names the net of U1.93 (PB7)
- net USART2_RX: no longer names the net of U1.87 (PD6)
- net USART2_TX: no longer names the net of U1.86 (PD5)
- new net: Q1.2 (G1), R35.2
- new net: Q1.4 (G2), R36.2
- new net: CN1.1, Q1.5 (D2), Q1.6 (D2)
- new net: CN1.3, Q1.7 (D1), Q1.8 (D1)
- new net: C36.1, U10.1 (IN), U10.3 (EN), U11.1 (K), U12.1 (K)
- new net: Q2.2 (G1), R37.2
- new net: Q2.4 (G2), R38.2
- new net: CN2.2, Q2.5 (D2), Q2.6 (D2)
- new net: CN2.4, Q2.7 (D1), Q2.8 (D1)
- new net: BUZZER1.1 (+), Q3.5 (D2), Q3.6 (D2), R30.1
- new net: BUZZER1.2, C33.1, R30.2
- new net FIRE_B: R2.1, R36.1, U1.30 (PA5)
- new net MMC_INT: U1.61 (PD14)
- no-connect marks 6 -> 10
Other:
- note added: "3.3V LDO"
- note added: "5V Buck (TPS62901RPJR set for vset mode)"
- note added: "Beeper"
- note added: "Companion UART"
- note added: "Pyro"
- note added: "Telemetry UART"
- note added: "VSET Mode, Output discharge YES, Auto PFM/PWM"
- note removed: "5V Buck"
- moved on the sheet: R15, R16

Commit message: Layout V1
Parts:
- removed C15: 100nF, PCM_JLCPCB:C_0402, symbol PCM_JLCPCB-Capacitors:0402,100nF
- added H1, H2, H3, H4: MountingHole_Pad_MP, MountingHole:MountingHole_3.2mm_M3_DIN965_Pad_TopBottom, symbol Mechanical:MountingHole_Pad_MP
Connections:
- net eMMC_CMD is gone; now on net SDMMC_CMD: R13.1
- net +3V3: now also J4.P4 (VDD)
- net FIRE_A: now also U1.33 (PC4); no longer U1.29 (PA4)
- net FIRE_B: now also U1.32 (PA7); no longer U1.30 (PA5)
- net FIRE_C: now also U1.30 (PA5); no longer U1.31 (PA6)
- net FIRE_D: now also U1.29 (PA4); no longer U1.32 (PA7)
- net GND: now also H1.1, H2.1, H3.1, H4.1
- net ICM_INT_2: no longer names the net of U1.42 (PE11)
Other:
- moved on the sheet: J7, J8

Commit message: Update
Parts:
- removed J4: MEM2080-00-128-00-A_REVA, SDholder:CONN_MEM2080-00-128-00-A_GCT, symbol MEM2080-00-128-00-A_REVA:MEM2080-00-128-00-A_REVA
- removed R5: 22Ω, PCM_JLCPCB:R_0402, symbol PCM_JLCPCB-Resistors:0402,22Ω
- removed R8: 1MΩ, PCM_JLCPCB:R_0402, symbol PCM_JLCPCB-Resistors:0402,1MΩ
- added Card1: TF-015, EasyEDA:TF-SMD_TF-015, symbol EasyEDA:TF-015
- added J2, J3: Conn_01x02_Pin, Connector_Molex:Molex_Micro-Fit_3.0_43650-0215_1x02_P3.00mm_Vertical, symbol Connector:Conn_01x02_Pin
- added JP1: Jumper_2_Bridged, Diode_SMD:D_0805_2012Metric, symbol Jumper:Jumper_2_Bridged
- J7: footprint Connector_PinHeader_2.54mm:PinHeader_1x04_P2.54mm_Vertical -> 1x04Molex:CONN_SD-43045-010_04_MOL
Connections:
- net SWO is gone; now on net DAT2: U1.89 (PB3)
- net +3V3: now also Card1.4 (VDD)
- net ADXL_INT1: no longer U1.77 (PA15)
- net Beeper: no longer U1.67 (PA8)
- net DAT0: now also U1.53 (PB14), Card1.7 (DAT0(D0)); no longer U1.65 (PC8)
- net DAT1: now also U1.54 (PB15), Card1.8 (DAT1(RSV)); no longer U1.66 (PC9)
- net DAT2: now also Card1.1 (DAT2(RSV)); no longer U1.78 (PC10)
- net DAT3: now also U1.90 (PB4), Card1.2 (CDDAT3(CS)); no longer U1.79 (PC11)
- net FIRE_A: now also U1.26 (PA3); no longer U1.33 (PC4)
- net FIRE_B: now also U1.25 (PA2); no longer U1.32 (PA7)
- net FIRE_C: now also U1.9 (PC15); no longer U1.30 (PA5)
- net FIRE_D: now also U1.8 (PC14); no longer U1.29 (PA4)
- net GND: now also J7.2 (Pin_2), Card1.10 (GND), Card1.11 (GND), Card1.12 (GND), Card1.13 (GND), Card1.6 (VSS), J2.1 (Pin_1), J3.1 (Pin_1), JP1.2 (B); no longer J7.4 (Pin_4), Q1.1 (S1), Q1.3 (S2), Q2.1 (S1), Q2.3 (S2)
- net ICM_CS: no longer U1.47 (PB10)
- net ICM_INT_1: no longer U1.41 (PE10)
- net MMC_INT: no longer U1.61 (PD14)
- net MS5607_CS: now also U1.67 (PA8); no longer U1.91 (PB5)
- net SDMMC_CLK: now also U1.87 (PD6), Card1.5 (CLK(SCLK)); no longer U1.80 (PC12)
- net SDMMC_CMD: now also U1.88 (PD7), Card1.3 (CMD(DI)); no longer U1.83 (PD2)
- net SPI1_MISO: now also U1.31 (PA6); no longer U1.45 (PE14)
- net SPI1_MOSI: now also U1.32 (PA7); no longer U1.46 (PE15)
- net SPI1_SCLK: now also U1.30 (PA5); no longer U1.44 (PE13)
- net UART4_RX: no longer U1.24 (PA1)
- net UART4_TX: no longer U1.23 (PA0)
- net USART1_RX: now also J7.4 (Pin_4), U1.68 (PA9); no longer J7.2 (Pin_2), U1.69 (PA10)
- net USART1_TX: now also U1.69 (PA10); no longer U1.68 (PA9)
- net USART3_RX: no longer U1.55 (PD8)
- net USART3_TX: no longer U1.56 (PD9)
- net VBAT+: no longer CN1.2, CN1.4, CN2.1, CN2.3
- net PYRO+: now reaches C31.1, C32.1, D3.2, J6.1
- net PYRO+: now also CN1.2, CN1.4, CN2.1, CN2.3
- net PWM1: now reaches U1.40 (PE9)
- net PWM1: now also J2.2 (Pin_2)
- net PWM2: now reaches U1.42 (PE11)
- net PWM2: now also J3.2 (Pin_2)
- new net PYRO_GND: JP1.1 (A), Q1.1 (S1), Q1.3 (S2), Q2.1 (S1), Q2.3 (S2)
- no-connect marks 10 -> 9
Other:
- moved on the sheet: C31, C32, CN1, CN2, D3, J6

Commit message: Final Layout (Pre-silkscreen)
- Added  1M resistors in parallel with the igniters for static dissipation
Parts:
- removed C10: 1uF, PCM_JLCPCB:C_0402, symbol PCM_JLCPCB-Capacitors:0402,1uF
- removed C11: 100pF, PCM_JLCPCB:C_0402, symbol PCM_JLCPCB-Capacitors:0402,100pF
- removed C31: 10uF, PCM_JLCPCB:C_0603, symbol PCM_JLCPCB-Capacitors:0603,10uF
- added C10, C11, C15: 100nF, PCM_JLCPCB:C_0402, symbol PCM_JLCPCB-Capacitors:0402,100nF
- added C25: 10uF, PCM_JLCPCB:C_0603, symbol PCM_JLCPCB-Capacitors:0402,10uF
- added C31: 10uF, PCM_JLCPCB:C_0603, symbol PCM_JLCPCB-Capacitors:0603,10uF,(2)
- added C37: 100nF, PCM_JLCPCB:C_0603, symbol PCM_JLCPCB-Capacitors:0603,100nF
- added D4: GREEN, LEDDD:WL-SMCW_0603, symbol Device:LED
- added D5: Blue, LEDDD:WL-SMCW_0603, symbol Device:LED
- added R19: 10kΩ, PCM_JLCPCB:R_0402, symbol PCM_JLCPCB-Resistors:0402,10kΩ
- added R20: 100Ω, PCM_JLCPCB:R_0402, symbol PCM_JLCPCB-Resistors:0402,100Ω
- added R21, R39: 470Ω, PCM_JLCPCB:R_0402, symbol PCM_JLCPCB-Resistors:0402,470Ω
- added R40, R41, R42, R43: 1MΩ, PCM_JLCPCB:R_0805, symbol PCM_JLCPCB-Resistors:0805,1MΩ
- added R5, R8: 75Ω, PCM_JLCPCB:R_0402, symbol PCM_JLCPCB-Resistors:0402,75Ω
- added U7: SN74AHCT125DR, EASYEDA:SOIC-14_L8.7-W3.9-P1.27-LS6.0-BL, symbol EasyEDA:SN74AHCT125DR
- added Y1: ECS-327TXO-33-TR, LSE:OSC_ECS-327TXO-33-TR, symbol ECS-327TXO-33-TR:ECS-327TXO-33-TR
- BUZZER1: footprint EasyEDA:BUZ-TH_BD14.0-P5.00-D0.7-FD -> EASYEDA:BUZ-TH_BD14.0-P5.00-D0.7-FD; Aliexpress (none) -> -; Digikey Part No. (none) -> 445-5242-1-ND; LCSC (none) -> -
- C1, C26, C35, C36: footprint PCM_JLCPCB:C_0402 -> PCM_JLCPCB:C_0603; Aliexpress (none) -> -; Digikey Part No. (none) -> -; LCSC C15525 -> C96446; Voltage Rated 6.3V -> 25V
- C12, C13, C14, C2, C27, C29, C3, C30, C32, C33, C4, C5, C6, C7, C8, C9, J5, R15, R16, R2, R22, R23, R26, R27, R28, R29, R3, R30, R32, R33, R34, R35, R36, R37, R38, R4: Aliexpress (none) -> -; Digikey Part No. (none) -> -
- C28: footprint PCM_JLCPCB:C_0603 -> PCM_JLCPCB:C_0805; Aliexpress (none) -> -; Digikey Part No. (none) -> -; LCSC C59461 -> C380338; Voltage Rated 6.3V -> 10V
- C34: footprint PCM_JLCPCB:C_0402 -> PCM_JLCPCB:C_0805; Aliexpress (none) -> -; Digikey Part No. (none) -> -; LCSC C23733 -> C76639
- CN1, CN2: footprint EasyEDA:CONN-TH_4P-P5.08_PA001-4P -> EASYEDA:CONN-TH_4P-P5.08_PA001-4P; Aliexpress (none) -> -; Digikey Part No. (none) -> -; LCSC (none) -> C173286
- Card1: footprint EasyEDA:TF-SMD_TF-015 -> EASYEDA:TF-SMD_TF-015; Aliexpress (none) -> -; Digikey Part No. (none) -> -; LCSC (none) -> C113206
- D1: footprint EasyEDA:SOT-23-6_L2.9-W1.6-P0.95-LS2.8-BL -> EASYEDA:SOT-23-6_L2.9-W1.6-P0.95-LS2.8-BL; Aliexpress (none) -> -; Digikey Part No. (none) -> 497-5235-1-ND; LCSC (none) -> -
- D2: value 3V 500mW -> MMSZ4683T1G; footprint EasyEDA:SOD-123_L2.8-W1.8-LS3.7-RD -> EASYEDA:SOD-123_L2.8-W1.8-LS3.7-RD; Aliexpress (none) -> -; Digikey Part No. (none) -> MMSZ4683T1GOSCT-ND; LCSC (none) -> -
- D3: footprint EasyEDA:SMA_L4.4-W2.6-LS5.0-RD -> EASYEDA:SMA_L4.4-W2.6-LS5.0-RD; Aliexpress (none) -> -; Digikey Part No. (none) -> -; LCSC (none) -> C466502
- FB1: Aliexpress (none) -> -; Digikey Part No. (none) -> -; LCSC (none) -> -; now left out of the parts list
- H1, H2, H3, H4, J1: Aliexpress (none) -> -; Digikey Part No. (none) -> -; LCSC (none) -> -
- J2, J3: Aliexpress (none) -> -; Digikey Part No. (none) -> WM1917-ND; LCSC (none) -> -
- J6: Aliexpress (none) -> -; Digikey Part No. (none) -> WM1865-ND; LCSC (none) -> -
- J7, J8: Aliexpress (none) -> -; Digikey Part No. (none) -> WM10667-ND; LCSC (none) -> -; now left out of the parts list
- JP1: Aliexpress (none) -> -; Digikey Part No. (none) -> 36-5106CT-ND; LCSC (none) -> -
- L1: footprint EasyEDA:IND-SMD_L4.0-W4.0 -> EASYEDA:IND-SMD_L4.0-W4.0; Aliexpress (none) -> -; Digikey Part No. (none) -> -; LCSC (none) -> C354573
- Q1, Q2, Q3: footprint EasyEDA:POWER-1212-8_L3.3-W3.3-P0.66-LS3.3-BL -> EASYEDA:POWER-1212-8_L3.3-W3.3-P0.66-LS3.3-BL; Aliexpress (none) -> -; Digikey Part No. (none) -> SI7232DN-T1-GE3CT-ND; LCSC (none) -> -
- R1, R10, R11, R12, R13, R9: Aliexpress (none) -> -; Digikey Part No. (none) -> 311-10.0KLRCT-ND; LCSC C25744 -> C25744 (OUT OF STOCK)
- R24: Aliexpress (none) -> -; Digikey Part No. (none) -> 311-76.8KHRCT-ND; LCSC C4124548 -> -
- R25: Aliexpress (none) -> -; Digikey Part No. (none) -> 311-26.1KHRCT-ND
- R7: Aliexpress (none) -> -; Digikey Part No. (none) -> 311-100KLRCT-ND (Alternatives); LCSC C25741 -> C25741 (OUT OF STOCK)
- SW1, SW2: footprint EasyEDA:SW-SMD_L3.9-W3.0-P4.45 -> EASYEDA:SW-SMD_L3.9-W3.0-P4.45; Aliexpress (none) -> -; Digikey Part No. (none) -> 4809-SKRKAEE020CT-ND; LCSC (none) -> -
- U1: Aliexpress (none) -> -; Digikey Part No. (none) -> 497-STM32U575VGT6-ND; LCSC (none) -> -
- U10: Aliexpress (none) -> -; Digikey Part No. (none) -> 296-50414-1-ND; LCSC (none) -> -
- U11, U12: footprint EasyEDA:SOD-123_L2.7-W1.6-LS3.7-RD-1 -> EASYEDA:SOD-123_L2.7-W1.6-LS3.7-RD-1; Aliexpress (none) -> -; Digikey Part No. (none) -> NRVB120VLSFT1GOSCT-ND; LCSC (none) -> -
- U2: footprint QFN_902RPJR_TEX -> TPSnew:QFN_902RPJR_TEX; Aliexpress (none) -> -; Digikey Part No. (none) -> 296-TPS62901RPJRCT-ND; LCSC (none) -> -
- X1: footprint EasyEDA:OSC-SMD_4P-L2.0-W1.6-BL_1XXD -> EASYEDA:OSC-SMD_4P-L2.0-W1.6-BL_1XXD; Aliexpress (none) -> -; Digikey Part No. (none) -> -; LCSC (none) -> C253694
Connections:
- net +3V3: now also SW2.2, C10.1, C11.1, C37.1, R20.1, R21.2, Y1.1 (OE), Y1.4 (SUPPLY_VOLTAGE); no longer J1.1 (VCC), SW2.1
- net +5V: now also C15.1, C25.1, U7.10 (~{3OE}), U7.13 (~{4OE}), U7.14 (VCC)
- net BAT_LEVEL: now also U1.18 (PC3); no longer U1.15 (PC0)
- net FIRE_D: now also U1.7 (PC13); no longer U1.8 (PC14)
- net GND: now also J5.A12B1 (GND), J5.B12A1 (GND), C10.2, C11.2, C15.2, C25.2, C31.2, C37.2, D4.1 (K), D5.1 (K), R19.2, U7.1 (~{1OE}), U7.12 (4A), U7.4 (~{2OE}), U7.7 (GND), U7.9 (3A), Y1.2 (GND); no longer SW2.2, U1.94 (PH3)
- net HSE_IN: now also X1.3 (Output)
- net ICM_CS: now also U1.37 (PB2)
- net MMC_INT: now also U1.52 (PB13)
- net PWM1: now also U7.2 (1A); no longer J2.2 (Pin_2)
- net PWM2: now also U7.5 (2A); no longer J3.2 (Pin_2)
- net PYRO+: now also C31.1, R40.1, R41.1, R42.1, R43.1
- net at CN1.1, Q1.5 (D2), Q1.6 (D2): now also R41.2
- net at CN1.3, Q1.7 (D1), Q1.8 (D1): now also R40.2
- net at CN2.2, Q2.5 (D2), Q2.6 (D2): now also R42.2
- net at CN2.4, Q2.7 (D1), Q2.8 (D1): now also R43.2
- net PA15: now reaches U1.77 (PA15)
- net PA15: now also R39.2
- new net: D4.2 (A), R21.1
- new net: D5.2 (A), R39.1
- new net: J1.1 (VCC), R20.2
- new net: R5.2, U7.3 (1Y)
- new net: R8.2, U7.6 (2Y)
- new net Boot0: R19.1, SW2.1, U1.94 (PH3)
- new net LSE_IN: U1.8 (PC14), Y1.3 (OUTPUT)
- new net SERVO1: J2.2 (Pin_2), R5.1
- new net SERVO2: J3.2 (Pin_2), R8.1
- no-connect marks 9 -> 12
Other:
- note added: "3OE and 4OE disabled"
- note added: "LSE 32.7680 kHz"
- note added: "PWM Level Shifting"
- note added: "Switch R35 to 220 Ohm if turn-on time too high"
- moved on the sheet: BUZZER1, C33, CN1, CN2, J2, J3, Q1, Q2, Q3, R2, R29, R30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
